Commit message: fixed the gazebo sim

File: tamiyabot_description/urdf/depth_camera.xacro (robot description, xacro)
@@ -1,49 +1,59 @@
-<?xml version="1.0"?>
-<robot xmlns:xacro="http://www.ros.org/wiki/xacro" >
+<?xml version="1.0" ?>
+<sdf version="1.6">
+  <model name="camera_model">
+    <link name="base_link">
+      <visual name="base_visual">
+        <geometry>
+          <box>
+            <size>0.1 0.1 0.1</size>
+          </box>
+        </geometry>
+        <material>
+          <ambient>0.2 0.2 0.2 1</ambient>
+        </material>
+      </visual>
+    </link>
+    <!-- Camera Link -->
+    <link name="camera_link">
+      <pose>0.13 0 0.2 0 0 0</pose>
+      <visual name="camera_visual">
+        <geometry>
+          <box>
+            <size>0.01 0.03 0.03</size>
+          </box>
+        </geometry>
+        <material>
+          <ambient>1 0 0 1</ambient>
+        </material>
+      </visual>
+    </link>
+    <!-- Fixed Joint -->
     <joint name="camera_joint" type="fixed">
-        <parent link="base_link"/>
-        <child link="camera_link"/>
-        <origin xyz="0.13 0 0.2" rpy="0 0 0"/>
+      <parent>base_link</parent>
+      <child>camera_link</child>
     </joint>
-    <link name="camera_link">
-        <visual>
-            <geometry>
-                <box size="0.010 0.03 0.03"/>
-            </geometry>
-            <material>
-                <color rgba="1 0 0 1"/>
-            </material>
-        </visual>
-    </link>
-    <joint name="camera_optical_joint" type="fixed">
-        <parent link="camera_link"/>
-        <child link="camera_link_optical"/>
-        <origin xyz="0 0 0" rpy="${-pi/2} 0 ${-pi/2}"/>
-    </joint>
-    <link name="camera_link_optical"></link>
-    <gazebo reference="camera_link">
-        <material>Gazebo/Red</material>
-        <sensor name="camera" type="depth">
-            <pose> 0 0 0 0 0 0 </pose>
-            <visualize>true</visualize>
-            <update_rate>10</update_rate>
-            <camera>
-                <horizontal_fov>1.089</horizontal_fov>
-                <image>
-                    <format>B8G8R8</format>
-                    <width>640</width>
-                    <height>480</height>
-                </image>
-                <clip>
-                    <near>0.05</near>
-                    <far>8.0</far>
-                </clip>
-            </camera>
-            <plugin name="camera_controller" filename="libgazebo_ros_camera.so">
-                <frame_name>camera_link_optical</frame_name>
-                <min_depth>0.05</min_depth>
-                <max_depth>100.0</max_depth>
-            </plugin>
-        </sensor>
-    </gazebo>
-</robot>
+    <!-- Camera Sensor -->
+    <sensor name="camera_sensor" type="depth">
+      <pose>0 0 0 0 0 0</pose>
+      <camera>
+        <horizontal_fov>1.089</horizontal_fov>
+        <image>
+          <width>640</width>
+          <height>480</height>
+          <format>B8G8R8</format>
+        </image>
+        <clip>
+          <near>0.05</near>
+          <far>8.0</far>
+        </clip>
+      </camera>
+      <plugin name="ros2_camera" filename="ignition-gazebo-camera-system">
+        <ros>
+          <namespace>/camera</namespace>
+          <remapping>image_raw:=/camera/image_raw</remapping>
+          <remapping>camera_info:=/camera/camera_info</remapping>
+        </ros>
+      </plugin>
+    </sensor>
+  </model>
+</sdf>

File: tamiyabot_description/urdf/ros2_controller.xacro (robot description, xacro)
@@ -1,28 +1,11 @@
 <?xml version="1.0"?>
-<robot xmlns:xacro="http://www.ros.org/wiki/xacro" name="bumperbot">
-    <gazebo reference="base_link">
-        <material>Gazebo/yellow</material>
-    </gazebo>
-    <xacro:macro name="wheel_gazebo" params="prefix">
-        <gazebo reference="${prefix}">
-            <material>Gazebo/Grey</material>
-        </gazebo>
-    </xacro:macro>
-    <xacro:wheel_gazebo prefix="front_left_wheel" />
-    <xacro:wheel_gazebo prefix="front_right_wheel" />
-    <xacro:wheel_gazebo prefix="rear_left_wheel" />
-    <xacro:wheel_gazebo prefix="rear_right_wheel" />
-    <gazebo reference="base_link">
-            <material>Gazebo/Yellow</material>
-    </gazebo>
+<robot xmlns:xacro="http://www.ros.org/wiki/xacro" name="tamiyabot">
      <!-- Ackermann driver -->
-  <ros2_control name="GazeboSystem" type="system">
+  <ros2_control name="RobotSystem" type="system">
         <!-- ros2_control Gazebo -->
         <xacro:if value="$(arg is_sim)">
-            <gazebo>
-                <plugin name="gazebo_ros2_control" filename="libgazebo_ros2_control.so">
-                    <parameters>$(find tamiyabot_controller)/config/tamiyabot_controllers.yaml</parameters>
-                </plugin>
-            </gazebo>
+            <hardware>
+                <plugin>gz_ros2_control/GazeboSimSystem</plugin>
+            </hardware>
         </xacro:if>
         <!-- ros2_control Real Robot -->
@@ -33,35 +16,35 @@
             </hardware>
         </xacro:unless>
-    <joint name="rear_left_wheel_joint">
-      <command_interface name="velocity"/>
-      <state_interface name="position"/>
-      <state_interface name="velocity"/>
-    </joint>
-    <joint name="rear_right_wheel_joint">
-      <command_interface name="velocity"/>
-      <state_interface name="position"/>
-      <state_interface name="velocity"/>
-    </joint>
-    <joint name="front_left_steering_joint">
-      <command_interface name="position"/>
-      <state_interface name="position"/>
-      <state_interface name="velocity"/>
-    </joint>
-    <joint name="front_right_steering_joint">
-      <command_interface name="position"/>
-      <state_interface name="position"/>
-      <state_interface name="velocity"/>
-    </joint>
-    <!--FRONT WHEEL-->
-    <joint name="front_left_wheel_joint">
-      <state_interface name="position"/>
-      <state_interface name="velocity"/>
-      <state_interface name="effort"/>
-    </joint>
-    <joint name="front_right_wheel_joint">
-      <state_interface name="position"/>
-      <state_interface name="velocity"/>
-      <state_interface name="effort"/>
-    </joint>
-  </ros2_control>
+      <joint name="rear_left_wheel_joint">
+        <command_interface name="velocity"/>
+        <state_interface name="position"/>
+        <state_interface name="velocity"/>
+      </joint>
+      <joint name="rear_right_wheel_joint">
+        <command_interface name="velocity"/>
+        <state_interface name="position"/>
+        <state_interface name="velocity"/>
+      </joint>
+      <joint name="front_left_steering_joint">
+        <command_interface name="position"/>
+        <state_interface name="position"/>
+        <state_interface name="velocity"/>
+      </joint>
+      <joint name="front_right_steering_joint">
+        <command_interface name="position"/>
+        <state_interface name="position"/>
+        <state_interface name="velocity"/>
+      </joint>
+      <!--FRONT WHEEL-->
+      <joint name="front_left_wheel_joint">
+        <state_interface name="position"/>
+        <state_interface name="velocity"/>
+        <state_interface name="effort"/>
+      </joint>
+      <joint name="front_right_wheel_joint">
+        <state_interface name="position"/>
+        <state_interface name="velocity"/>
+        <state_interface name="effort"/>
+      </joint>
+    </ros2_control>
 </robot>

File: tamiyabot_description/urdf/tamiyabot.urdf.xacro (robot description, xacro)
@@ -1,7 +1,9 @@
 <?xml version="1.0"?>
 <robot name="tamiyabot" xmlns:xacro="http://www.ros.org/wiki/xacro">
-    <xacro:include filename="$(find tamiyabot_description)/urdf/tamiyabot_gazebo.xacro"/>
-    <!-- <xacro:include filename="$(find tamiyabot_description)/urdf/ros2_controller.xacro"/> -->
-    <xacro:include filename="$(find tamiyabot_description)/urdf/depth_camera.xacro"/>
+    <!-- Load Simulated or Real Hardware Interfaces -->
+    <xacro:arg name="is_sim" default="true"/>
+    <!-- <xacro:include filename="$(find tamiyabot_description)/urdf/tamiyabot_gazebo.xacro"/>
+    <xacro:include filename="$(find tamiyabot_description)/urdf/ros2_controller.xacro"/> -->
+    <!-- <xacro:include filename="$(find tamiyabot_description)/urdf/depth_camera.xacro"/> -->
     <material name="white">
         <color rgba="1 1 1 1"/>
@@ -194,4 +196,5 @@
         <origin xyz="-0.127 0.077 ${wheel_down}" rpy="0.0 0.0 0.0"/>
         <axis xyz="0 1 0"/>
+        <dynamics damping="0.2" />
     </joint>
     <joint name="rear_right_wheel_joint" type="continuous">
@@ -200,4 +203,5 @@
         <origin xyz="-0.127 -0.077 ${wheel_down}" rpy="0.0 0.0 0.0"/>
         <axis xyz="0 1 0"/>
+        <dynamics damping="0.2" />
     </joint>
     <!-- front wheel joints -->
@@ -207,4 +211,5 @@
         <origin xyz="0.0 0.00 ${wheel_down}" rpy="0.0 0.0 0.0"/>
         <axis xyz="0 1 0"/>
+        <dynamics damping="0.2" />
     </joint>
     <joint name="front_right_wheel_joint" type="continuous">
@@ -213,4 +218,33 @@
         <origin xyz="0.0 0.00 ${wheel_down}" rpy="0.0 0.0 0.0"/>
         <axis xyz="0 1 0"/>
-    </joint>
+        <dynamics damping="0.2" />
+    </joint>
+     <ros2_control name="GazeboSystem" type="system">
+    <hardware>
+      <plugin>gz_ros2_control/GazeboSimSystem</plugin>
+    </hardware>
+    <joint name="rear_left_wheel_joint">
+      <command_interface name="velocity" />
+      <state_interface name="velocity" />
+      <state_interface name="position" />
+    </joint>
+    <joint name="rear_right_wheel_joint">
+      <command_interface name="velocity" />
+      <state_interface name="velocity" />
+      <state_interface name="position" />
+    </joint>
+    <joint name="front_left_steering_joint">
+      <command_interface name="position" />
+      <state_interface name="position" />
+    </joint>
+    <joint name="front_right_steering_joint">
+      <command_interface name="position" />
+      <state_interface name="position" />
+    </joint>
+  </ros2_control>
+      <gazebo>
+    <plugin filename="gz_ros2_control-system" name="gz_ros2_control::GazeboSimROS2ControlPlugin">
+      <parameters>$(find tamiyabot_controller)/config/tamiyabot_controllers.yaml</parameters>
+    </plugin>
+  </gazebo>
 </robot>

File: tamiyabot_description/urdf/tamiyabot_gazebo.xacro (robot description, xacro)
@@ -1,61 +1,87 @@
 <?xml version="1.0"?>
-<robot xmlns:xacro="http://www.ros.org/wiki/xacro">
-    <gazebo reference="base_link">
-        <material>Gazebo/yellow</material>
+<robot xmlns:xacro="http://www.ros.org/wiki/xacro" xmlns:ign="http://ignitionrobotics.org/schemas">
+    <!-- Ignition Gazebo material for the base -->
+    <ign:model>
+        <link name="base_link">
+            <visual>
+                <material>Gazebo/Yellow</material>
+            </visual>
+        </link>
+    </ign:model>
+    <!-- XACRO macro for setting wheel materials in Ignition Gazebo -->
+    <xacro:macro name="wheel_ignition" params="prefix">
+        <ign:model>
+            <link name="${prefix}">
+                <visual>
+                    <material>Gazebo/Grey</material>
+                </visual>
+            </link>
+        </ign:model>
+    </xacro:macro>
+    <!-- Apply wheel Ignition Gazebo materials -->
+    <xacro:wheel_ignition prefix="front_left_wheel" />
+    <xacro:wheel_ignition prefix="front_right_wheel" />
+    <xacro:wheel_ignition prefix="rear_left_wheel" />
+    <xacro:wheel_ignition prefix="rear_right_wheel" />
+    <gazebo reference="front_left_wheel">
+        <mu1>1000000000000000.0</mu1>
+        <mu2>1000000000000000.0</mu2>
+        <kp>1000000000000.0</kp>
+        <kd>10.0</kd>
+        <minDepth>0.001</minDepth>
+        <maxVel>0.1</maxVel>
+        <fdir1>1 0 0</fdir1>
     </gazebo>
-    <xacro:macro name="wheel_gazebo" params="prefix">
-        <gazebo reference="${prefix}">
-            <material>Gazebo/Grey</material>
-        </gazebo>
-    </xacro:macro>
-    <xacro:wheel_gazebo prefix="front_left_wheel" />
-    <xacro:wheel_gazebo prefix="front_right_wheel" />
-    <xacro:wheel_gazebo prefix="rear_left_wheel" />
-    <xacro:wheel_gazebo prefix="rear_right_wheel" />
-    <gazebo reference="base_link">
-            <material>Gazebo/Yellow</material>
+    <gazebo reference="front_right_wheel">
+        <mu1>1000000000000000.0</mu1>
+        <mu2>1000000000000000.0</mu2>
+        <kp>1000000000000.0</kp>
+        <kd>10.0</kd>
+        <minDepth>0.001</minDepth>
+        <maxVel>0.1</maxVel>
+        <fdir1>1 0 0</fdir1>
     </gazebo>
-    <!-- <xacro:wheel_gazebo prefix="steering" />-->
-     <!-- Ackermann driver -->
-  <ros2_control name="GazeboSystem" type="system">
-    <hardware>
-      <plugin>gazebo_ros2_control/GazeboSystem</plugin>
-    </hardware>
-    <joint name="rear_left_wheel_joint">
-      <command_interface name="velocity"/>
-      <state_interface name="position"/>
-      <state_interface name="velocity"/>
-    </joint>
-    <joint name="rear_right_wheel_joint">
-      <command_interface name="velocity"/>
-      <state_interface name="position"/>
-      <state_interface name="velocity"/>
-    </joint>
-    <joint name="front_left_steering_joint">
-      <command_interface name="position"/>
-      <state_interface name="position"/>
-      <state_interface name="velocity"/>
-    </joint>
-    <joint name="front_right_steering_joint">
-      <command_interface name="position"/>
-      <state_interface name="position"/>
-      <state_interface name="velocity"/>
-    </joint>
-    <!--FRONT WHEEL-->
-    <joint name="front_left_wheel_joint">
-      <state_interface name="position"/>
-      <state_interface name="velocity"/>
-      <state_interface name="effort"/>
-    </joint>
-    <joint name="front_right_wheel_joint">
-      <state_interface name="position"/>
-      <state_interface name="velocity"/>
-      <state_interface name="effort"/>
-    </joint>
-  </ros2_control>
-  <gazebo>
-    <plugin name="gazebo_ros2_control" filename="libgazebo_ros2_control.so">
-        <parameters>$(find tamiyabot_controller)/config/tamiyabot_controllers.yaml</parameters>
-    </plugin>
-  </gazebo>
+    <gazebo reference="rear_left_wheel">
+        <mu1>1000000000000000.0</mu1>
+        <mu2>1000000000000000.0</mu2>
+        <kp>1000000000000.0</kp>
+        <kd>10.0</kd>
+        <minDepth>0.001</minDepth>
+        <maxVel>0.1</maxVel>
+        <fdir1>1 0 0</fdir1>
+    </gazebo>
+    <gazebo reference="rear_right_wheel">
+        <mu1>1000000000000000.0</mu1>
+        <mu2>1000000000000000.0</mu2>
+        <kp>1000000000000.0</kp>
+        <kd>10.0</kd>
+        <minDepth>0.001</minDepth>
+        <maxVel>0.1</maxVel>
+        <fdir1>1 0 0</fdir1>
+    </gazebo>
+    <!-- Ignition Gazebo material for the base again (if needed) -->
+    <ign:model>
+        <link name="base_link">
+            <visual>
+                <material>Gazebo/Yellow</material>
+            </visual>
+        </link>
+    </ign:model>
+    <gazebo>
+        <plugin filename="gz-sim-joint-state-publisher-system" name="gz::sim::systems::JointStatePublisher">
+            <topic>joint_states</topic>
+            <joint_name>front_left_steering_joint</joint_name>
+            <joint_name>front_right_steering_joint</joint_name>
+            <joint_name>front_left_wheel_joint</joint_name>
+            <joint_name>front_right_wheel_joint</joint_name>
+            <joint_name>rear_left_wheel_joint</joint_name>
+            <joint_name>rear_right_wheel_joint</joint_name>
+        </plugin>
+        <plugin filename="gz_ros2_control-system" name="gz_ros2_control::GazeboSimROS2ControlPlugin">
+            <parameters>$(find tamiyabot_controller)/config/tamiyabot_controllers.yaml</parameters>
+        </plugin>
+        <plugin filename="gz-sim-sensors-system" name="gz::sim::systems::Sensors">
+            <render_engine>ogre2</render_engine>
+        </plugin>
+    </gazebo>
 </robot>
