Commit message: add lidar into gazebo

File: tamiyabot_description/urdf/camera.xacro (robot description, xacro)
@@ -7,5 +7,5 @@
         <parent link="base_link"/>
         <child link="camera_link"/>
-        <origin xyz="0.128 0 0.095" rpy="0 0 0"/>
+        <origin xyz="-0.1 0 0.095" rpy="0 0 0"/>
     </joint>
     <link name="camera_link">
@@ -23,6 +23,6 @@
     </joint>
     <link name="camera_link_optical"></link>
-    <gazebo reference="camera_link">
-        <material>Gazebo/Red</material>
+        <gazebo reference="camera_link">
+        <material>Gazebo/Black</material>
         <sensor name="camera" type="camera">
             <pose> 0 0 0 0 0 0 </pose>
@@ -30,4 +30,5 @@
             <update_rate>10</update_rate>
             <camera>
+                <camera_info_topic>camera/camera_info</camera_info_topic>
                 <horizontal_fov>1.089</horizontal_fov>
                 <image>
@@ -41,7 +42,6 @@
                 </clip>
             </camera>
-            <plugin name="camera_controller" filename="libgazebo_ros_camera.so">
-                <frame_name>camera_link_optical</frame_name>
-            </plugin>
+            <topic>camera/image_raw</topic>
+            <gz_frame_id>camera_link_optical</gz_frame_id>
         </sensor>
     </gazebo>

File: tamiyabot_description/urdf/depth_camera.xacro (robot description, xacro)
@@ -1,4 +1,4 @@
 <?xml version="1.0" ?>
-<sdf version="1.6">
+<sdf version="1.9">
   <model name="camera_model">
     <link name="base_link">
@@ -48,5 +48,5 @@
         </clip>
       </camera>
-      <plugin name="ros2_camera" filename="ignition-gazebo-camera-system">
+      <plugin name="ros2_camera" filename="libgazebo_ros_camera.so">
         <ros>
           <namespace>/camera</namespace>

File: tamiyabot_description/urdf/tamiyabot_gazebo.xacro (robot description, xacro)
@@ -5,4 +5,37 @@
             <parameters>$(find tamiyabot_controller)/config/tamiyabot_controllers.yaml</parameters>
         </plugin>
-  </gazebo>
+        <plugin filename="gz-sim-sensors-system" name="gz::sim::systems::Sensors">
+            <render_engine>ogre2</render_engine>
+        </plugin>
+    </gazebo>
+    <gazebo reference="laser_link">
+        <material>Gazebo/Black</material>
+        <sensor name="lidar" type="gpu_lidar">
+            <always_on>true</always_on>
+            <visualize>true</visualize>
+            <topic>scan</topic>
+            <update_rate>5</update_rate>
+            <gz_frame_id>laser_link</gz_frame_id>
+            <lidar>
+                <scan>
+                    <horizontal>
+                        <samples>360</samples>
+                        <resolution>1.00000</resolution>
+                        <min_angle>0.000000</min_angle>
+                        <max_angle>6.280000</max_angle>
+                    </horizontal>
+                </scan>
+                <range>
+                    <min>0.120000</min>
+                    <max>12.0</max>
+                    <resolution>0.02</resolution>
+                </range>
+                <noise>
+                    <type>gaussian</type>
+                    <mean>0.0</mean>
+                    <stddev>0.01</stddev>
+                </noise>
+            </lidar>
+        </sensor>
+    </gazebo>
 </robot>

File: tamiyabot_description/urdf/tamiyabot_model.urdf.xacro (robot description, xacro)
@@ -5,7 +5,11 @@
     <xacro:include filename="$(find tamiyabot_description)/urdf/tamiyabot_gazebo.xacro"/>
     <xacro:include filename="$(find tamiyabot_description)/urdf/ros2_controller.xacro"/>
-    <xacro:include filename="$(find tamiyabot_description)/urdf/depth_camera.xacro"/>
-    <material name="silver">
-      <color rgba="0.700 0.700 0.700 1.000"/>
+    <xacro:include filename="$(find tamiyabot_description)/urdf/camera.xacro"/>
+    <xacro:include filename="$(find tamiyabot_description)/urdf/lidar.xacro"/>
+    <material name="yellow">
+      <color rgba="0.700 0.700 0.0 1.000"/>
+    </material>
+    <material name="black">
+      <color rgba="0.0 0.0 0.0 1.000"/>
     </material>
     <link name="base_footprint"/>
@@ -21,5 +25,5 @@
           <mesh filename="package://tamiyabot_description/meshes/base_link.stl" scale="0.001 0.001 0.001"/>
         </geometry>
-        <material name="silver"/>
+        <material name="yellow"/>
         <material/>
       </visual>
@@ -42,5 +46,5 @@
           <mesh filename="package://tamiyabot_description/meshes/rear_left_wheel1.stl" scale="0.001 0.001 0.001"/>
         </geometry>
-        <material name="silver"/>
+        <material name="black"/>
         <material/>
       </visual>
@@ -63,5 +67,5 @@
           <mesh filename="package://tamiyabot_description/meshes/rear_right_wheel1.stl" scale="0.001 0.001 0.001"/>
         </geometry>
-        <material name="silver"/>
+        <material name="black"/>
         <material/>
       </visual>
@@ -84,5 +88,5 @@
           <mesh filename="package://tamiyabot_description/meshes/front_left_wheel1.stl" scale="0.001 0.001 0.001"/>
         </geometry>
-        <material name="silver"/>
+        <material name="black"/>
         <material/>
       </visual>
@@ -105,5 +109,5 @@
           <mesh filename="package://tamiyabot_description/meshes/front_right_wheel1.stl" scale="0.001 0.001 0.001"/>
         </geometry>
-        <material name="silver"/>
+        <material name="black"/>
         <material/>
       </visual>
@@ -126,5 +130,5 @@
           <mesh filename="package://tamiyabot_description/meshes/steering_right_link1.stl" scale="0.001 0.001 0.001"/>
         </geometry>
-        <material name="silver"/>
+        <material name="black"/>
         <material/>
       </visual>
@@ -147,5 +151,5 @@
           <mesh filename="package://tamiyabot_description/meshes/steering_left_link1.stl" scale="0.001 0.001 0.001"/>
         </geometry>
-        <material name="silver"/>
+        <material name="black"/>
         <material/>
       </visual>
@@ -175,4 +179,18 @@
       <axis xyz="0.0 -1.0 0.0"/>
     </joint>
+    <joint name="front_right_steering_joint" type="revolute">
+      <origin xyz="-0.030009 -0.0685 -0.009" rpy="0 0 0"/>
+      <parent link="base_link"/>
+      <child link="steering_right_link1"/>
+      <axis xyz="0.0 0.0 -1.0"/>
+      <limit effort="1000.0" lower="-0.78" upper="0.78" velocity="30"/>
+    </joint>
+    <joint name="front_left_steering_joint" type="revolute">
+      <origin xyz="-0.030009 0.0685 -0.009" rpy="0 0 0"/>
+      <parent link="base_link"/>
+      <child link="steering_left_link1"/>
+      <axis xyz="0.0 0.0 -1.0"/>
+      <limit effort="1000.0" lower="-0.78" upper="0.78" velocity="30"/>
+    </joint>
     <joint name="front_right_wheel_joint" type="continuous">
       <origin xyz="0.0 0.0 -0.004" rpy="0 0 0"/>
@@ -187,17 +205,3 @@
       <axis xyz="0.0 1.0 0.0"/>
     </joint>
-    <joint name="front_right_steering_joint" type="revolute">
-      <origin xyz="-0.030009 -0.0685 -0.009" rpy="0 0 0"/>
-      <parent link="base_link"/>
-      <child link="steering_right_link1"/>
-      <axis xyz="0.0 0.0 -1.0"/>
-      <limit effort="1000.0" lower="-0.78" upper="0.78" velocity="30"/>
-    </joint>
-    <joint name="front_left_steering_joint" type="revolute">
-      <origin xyz="-0.030009 0.0685 -0.009" rpy="0 0 0"/>
-      <parent link="base_link"/>
-      <child link="steering_left_link1"/>
-      <axis xyz="0.0 0.0 -1.0"/>
-      <limit effort="1000.0" lower="-0.78" upper="0.78" velocity="30"/>
-    </joint>
 </robot>

Commit message: Create autonomous_drive package

File: tamiyabot_description/urdf/camera.xacro (robot description, xacro)
@@ -7,5 +7,5 @@
         <parent link="base_link"/>
         <child link="camera_link"/>
-        <origin xyz="-0.1 0 0.095" rpy="0 0 0"/>
+        <origin xyz="-0.1 0 0.095" rpy="0 0 3.14159"/>
     </joint>
     <link name="camera_link">
