Commit message: add to urdf to publish odom

File: tamiyabot_description/urdf/tamiyabot_gazebo.xacro (robot description, xacro)
@@ -3,4 +3,8 @@
     <gazebo>
         <plugin filename="gz_ros2_control-system" name="gz_ros2_control::GazeboSimROS2ControlPlugin">
+            <ros>
+                <remapping>tamiyabot_controller/odometry:=odom</remapping>
+                <remapping>tamiyabot_controller/tf_odometry:=tf</remapping>
+            </ros>
             <parameters>$(find tamiyabot_controller)/config/tamiyabot_controllers.yaml</parameters>
         </plugin>
@@ -8,4 +12,20 @@
             <render_engine>ogre2</render_engine>
         </plugin>
+    </gazebo>
+    <gazebo reference="front_right_wheel">
+        <mu1>1.0</mu1>
+        <mu2>1.0</mu2>
+    </gazebo>
+    <gazebo reference="front_left_wheel">
+        <mu1>1.0</mu1>
+        <mu2>1.0</mu2>
+    </gazebo>
+    <gazebo reference="rear_right_wheel">
+        <mu1>1.0</mu1>
+        <mu2>1.0</mu2>
+    </gazebo>
+    <gazebo reference="rear_left_wheel">
+        <mu1>1.0</mu1>
+        <mu2>1.0</mu2>
     </gazebo>
     <gazebo reference="laser_link">

File: tamiyabot_description/urdf/tamiyabot_model.urdf.xacro (robot description, xacro)
@@ -1,5 +1,6 @@
 <?xml version="1.0" ?>
 <robot name="tamiyabot" xmlns:xacro="http://www.ros.org/wiki/xacro">
-  <xacro:arg name="is_sim" default="true"/>
+  <!-- Load Simulated or Real Hardware Interfaces -->
+    <xacro:arg name="is_sim" default="true"/>
   <xacro:include filename="$(find tamiyabot_description)/urdf/tamiyabot_gazebo.xacro"/>
   <xacro:include filename="$(find tamiyabot_description)/urdf/ros2_controller.xacro"/>
@@ -99,5 +100,5 @@
 <link name="front_right_wheel1">
   <inertial>
-    <origin xyz="3.2111828563233247e-07 -0.01046581392999707 1.5959455978986625e-16" rpy="0 0 0"/>
+    <origin xyz="3.2111828563233247e-07 0.0 1.5959455978986625e-16" rpy="0 0 0"/>
     <mass value="0.9105437032741225"/>
     <inertia ixx="0.0004316099354611056" iyy="0.000796368727658819" izz="0.0004316121960988347" ixy="7.37257477290143e-18" iyz="2.168404344971009e-18" ixz="5.800481622797449e-18"/>
@@ -141,5 +142,5 @@
 <link name="front_left_wheel1">
   <inertial>
-    <origin xyz="3.2111828832809275e-07 0.010465813929997764 1.734723475976807e-18" rpy="0 0 0"/>
+    <origin xyz="3.2111828832809275e-07 0.0 1.734723475976807e-18" rpy="0 0 0"/>
     <mass value="0.9105437032741228"/>
     <inertia ixx="0.0004316099354611104" iyy="0.0007963687276588275" izz="0.00043161219609884295" ixy="7.37257477290143e-18" iyz="-1.0842021724855044e-19" ixz="-7.589415207398531e-19"/>
@@ -204,5 +205,5 @@
   <child link="steering_right_link1"/>
   <axis xyz="0.0 0.0 -1.0"/>
-  <limit upper="0.785398" lower="-0.785398" effort="100000" velocity="30"/>
+  <limit upper="0.785398" lower="-0.785398" effort="100" velocity="30"/>
 </joint>
 <joint name="front_left_steering_joint" type="revolute">
@@ -211,8 +212,8 @@
   <child link="steering_left_link1"/>
   <axis xyz="0.0 0.0 -1.0"/>
-  <limit upper="0.785398" lower="-0.785398" effort="100000" velocity="30"/>
+  <limit upper="0.785398" lower="-0.785398" effort="100" velocity="30"/>
 </joint>
 <joint name="front_right_wheel_joint" type="continuous">
-  <origin xyz="0.0 0.0 0.004" rpy="0 0 0"/>
+  <origin xyz="0.0 0.01 0.004" rpy="0 0 0"/>
   <parent link="steering_right_link1"/>
   <child link="front_right_wheel1"/>
@@ -220,5 +221,5 @@
 </joint>
 <joint name="front_left_wheel_joint" type="continuous">
-  <origin xyz="0.0 0.0 0.004" rpy="0 0 0"/>
+  <origin xyz="0.0 -0.01 0.004" rpy="0 0 0"/>
   <parent link="steering_left_link1"/>
   <child link="front_left_wheel1"/>
