Commit message: Create model and meshes and fixed the controller issue

File: tamiyabot_description/urdf/ros2_controller.xacro (robot description, xacro)
@@ -5,7 +5,25 @@
         <!-- ros2_control Gazebo -->
         <xacro:if value="$(arg is_sim)">
-            <hardware>
+              <hardware>
                 <plugin>gz_ros2_control/GazeboSimSystem</plugin>
-            </hardware>
+              </hardware>
+              <joint name="rear_left_wheel_joint">
+                <command_interface name="velocity" />
+                <state_interface name="velocity" />
+                <state_interface name="position" />
+              </joint>
+              <joint name="rear_right_wheel_joint">
+                <command_interface name="velocity" />
+                <state_interface name="velocity" />
+                <state_interface name="position" />
+              </joint>
+              <joint name="front_left_steering_joint">
+                <command_interface name="position" />
+                <state_interface name="position" />
+              </joint>
+              <joint name="front_right_steering_joint">
+                <command_interface name="position" />
+                <state_interface name="position" />
+              </joint>
         </xacro:if>
         <!-- ros2_control Real Robot -->
@@ -16,35 +34,4 @@
             </hardware>
         </xacro:unless>
-      <joint name="rear_left_wheel_joint">
-        <command_interface name="velocity"/>
-        <state_interface name="position"/>
-        <state_interface name="velocity"/>
-      </joint>
-      <joint name="rear_right_wheel_joint">
-        <command_interface name="velocity"/>
-        <state_interface name="position"/>
-        <state_interface name="velocity"/>
-      </joint>
-      <joint name="front_left_steering_joint">
-        <command_interface name="position"/>
-        <state_interface name="position"/>
-        <state_interface name="velocity"/>
-      </joint>
-      <joint name="front_right_steering_joint">
-        <command_interface name="position"/>
-        <state_interface name="position"/>
-        <state_interface name="velocity"/>
-      </joint>
-      <!--FRONT WHEEL-->
-      <joint name="front_left_wheel_joint">
-        <state_interface name="position"/>
-        <state_interface name="velocity"/>
-        <state_interface name="effort"/>
-      </joint>
-      <joint name="front_right_wheel_joint">
-        <state_interface name="position"/>
-        <state_interface name="velocity"/>
-        <state_interface name="effort"/>
-      </joint>
     </ros2_control>
 </robot>

File: tamiyabot_description/urdf/tamiyabot.urdf.xacro (robot description, xacro)
@@ -175,18 +175,14 @@
         <parent link="base_link"/>
         <child link="left_kingpin"/>
-        <origin xyz="0.145 0.077 0.0" rpy="0.0 0.0 0.0"/>
+        <origin xyz="0.145 0.077 ${wheel_down}" rpy="0.0 0.0 0.0"/>
         <axis xyz="0 0 1"/>
-        <limit effort="${steer_effort}"
-               lower="${steer_limit_deg * deg_to_rad * -1.0}" upper="${steer_limit_deg * deg_to_rad}"
-               velocity="${steer_velocity}"/>
+        <limit effort="1000.0" lower="-0.78" upper="0.78" velocity="30"/>
     </joint>
     <joint name="front_right_steering_joint" type="revolute">
         <parent link="base_link"/>
         <child link="right_kingpin"/>
-        <origin xyz="0.145 -0.077 0.0" rpy="0.0 0.0 0.0"/>
+        <origin xyz="0.145 -0.077 ${wheel_down}" rpy="0.0 0.0 0.0"/>
         <axis xyz="0 0 1"/>
-        <limit effort="${steer_effort}"
-               lower="${steer_limit_deg * deg_to_rad * -1.0}" upper="${steer_limit_deg * deg_to_rad}"
-               velocity="${steer_velocity}"/>
+        <limit effort="1000.0" lower="-0.78" upper="0.78" velocity="30"/>
     </joint>
     <!-- rear wheel joints -->
@@ -209,5 +205,5 @@
         <parent link="left_kingpin"/>
         <child link="front_left_wheel"/>
-        <origin xyz="0.0 0.00 ${wheel_down}" rpy="0.0 0.0 0.0"/>
+        <origin xyz="0.0 0.00 0.0" rpy="0.0 0.0 0.0"/>
         <axis xyz="0 1 0"/>
         <dynamics damping="0.2" />
@@ -216,35 +212,7 @@
         <parent link="right_kingpin"/>
         <child link="front_right_wheel"/>
-        <origin xyz="0.0 0.00 ${wheel_down}" rpy="0.0 0.0 0.0"/>
-        <axis xyz="0 1 0"/>
-        <dynamics damping="0.2" />
-    </joint>
-     <ros2_control name="GazeboSystem" type="system">
-    <hardware>
-      <plugin>gz_ros2_control/GazeboSimSystem</plugin>
-    </hardware>
-    <joint name="rear_left_wheel_joint">
-      <command_interface name="velocity" />
-      <state_interface name="velocity" />
-      <state_interface name="position" />
-    </joint>
-    <joint name="rear_right_wheel_joint">
-      <command_interface name="velocity" />
-      <state_interface name="velocity" />
-      <state_interface name="position" />
-    </joint>
-    <joint name="front_left_steering_joint">
-      <command_interface name="position" />
-      <state_interface name="position" />
-    </joint>
-    <joint name="front_right_steering_joint">
-      <command_interface name="position" />
-      <state_interface name="position" />
-    </joint>
-  </ros2_control>
-      <gazebo>
-    <plugin filename="gz_ros2_control-system" name="gz_ros2_control::GazeboSimROS2ControlPlugin">
-      <parameters>$(find tamiyabot_controller)/config/tamiyabot_controllers.yaml</parameters>
-    </plugin>
-  </gazebo>
+        <origin xyz="0.0 0.00 0.0" rpy="0.0 0.0 0.0"/>
+        <axis xyz="0 1 0"/>
+        <dynamics damping="0.2" />
+    </joint>
 </robot>

File: tamiyabot_description/urdf/tamiyabot_gazebo.xacro (robot description, xacro)
@@ -1,87 +1,8 @@
 <?xml version="1.0"?>
 <robot xmlns:xacro="http://www.ros.org/wiki/xacro" xmlns:ign="http://ignitionrobotics.org/schemas">
-    <!-- Ignition Gazebo material for the base -->
-    <ign:model>
-        <link name="base_link">
-            <visual>
-                <material>Gazebo/Yellow</material>
-            </visual>
-        </link>
-    </ign:model>
-    <!-- XACRO macro for setting wheel materials in Ignition Gazebo -->
-    <xacro:macro name="wheel_ignition" params="prefix">
-        <ign:model>
-            <link name="${prefix}">
-                <visual>
-                    <material>Gazebo/Grey</material>
-                </visual>
-            </link>
-        </ign:model>
-    </xacro:macro>
-    <!-- Apply wheel Ignition Gazebo materials -->
-    <xacro:wheel_ignition prefix="front_left_wheel" />
-    <xacro:wheel_ignition prefix="front_right_wheel" />
-    <xacro:wheel_ignition prefix="rear_left_wheel" />
-    <xacro:wheel_ignition prefix="rear_right_wheel" />
-    <gazebo reference="front_left_wheel">
-        <mu1>1000000000000000.0</mu1>
-        <mu2>1000000000000000.0</mu2>
-        <kp>1000000000000.0</kp>
-        <kd>10.0</kd>
-        <minDepth>0.001</minDepth>
-        <maxVel>0.1</maxVel>
-        <fdir1>1 0 0</fdir1>
-    </gazebo>
-    <gazebo reference="front_right_wheel">
-        <mu1>1000000000000000.0</mu1>
-        <mu2>1000000000000000.0</mu2>
-        <kp>1000000000000.0</kp>
-        <kd>10.0</kd>
-        <minDepth>0.001</minDepth>
-        <maxVel>0.1</maxVel>
-        <fdir1>1 0 0</fdir1>
-    </gazebo>
-    <gazebo reference="rear_left_wheel">
-        <mu1>1000000000000000.0</mu1>
-        <mu2>1000000000000000.0</mu2>
-        <kp>1000000000000.0</kp>
-        <kd>10.0</kd>
-        <minDepth>0.001</minDepth>
-        <maxVel>0.1</maxVel>
-        <fdir1>1 0 0</fdir1>
-    </gazebo>
-    <gazebo reference="rear_right_wheel">
-        <mu1>1000000000000000.0</mu1>
-        <mu2>1000000000000000.0</mu2>
-        <kp>1000000000000.0</kp>
-        <kd>10.0</kd>
-        <minDepth>0.001</minDepth>
-        <maxVel>0.1</maxVel>
-        <fdir1>1 0 0</fdir1>
-    </gazebo>
-    <!-- Ignition Gazebo material for the base again (if needed) -->
-    <ign:model>
-        <link name="base_link">
-            <visual>
-                <material>Gazebo/Yellow</material>
-            </visual>
-        </link>
-    </ign:model>
     <gazebo>
-        <plugin filename="gz-sim-joint-state-publisher-system" name="gz::sim::systems::JointStatePublisher">
-            <topic>joint_states</topic>
-            <joint_name>front_left_steering_joint</joint_name>
-            <joint_name>front_right_steering_joint</joint_name>
-            <joint_name>front_left_wheel_joint</joint_name>
-            <joint_name>front_right_wheel_joint</joint_name>
-            <joint_name>rear_left_wheel_joint</joint_name>
-            <joint_name>rear_right_wheel_joint</joint_name>
-        </plugin>
         <plugin filename="gz_ros2_control-system" name="gz_ros2_control::GazeboSimROS2ControlPlugin">
             <parameters>$(find tamiyabot_controller)/config/tamiyabot_controllers.yaml</parameters>
         </plugin>
-        <plugin filename="gz-sim-sensors-system" name="gz::sim::systems::Sensors">
-            <render_engine>ogre2</render_engine>
-        </plugin>
-    </gazebo>
+  </gazebo>
 </robot>

Commit message: modify the model to bicycle controller

File: tamiyabot_description/urdf/ros2_controller.xacro (robot description, xacro)
@@ -1,37 +1,30 @@
 <?xml version="1.0"?>
 <robot xmlns:xacro="http://www.ros.org/wiki/xacro" name="tamiyabot">
-     <!-- Ackermann driver -->
+  <!-- Ackermann driver -->
   <ros2_control name="RobotSystem" type="system">
-        <!-- ros2_control Gazebo -->
-        <xacro:if value="$(arg is_sim)">
-              <hardware>
-                <plugin>gz_ros2_control/GazeboSimSystem</plugin>
-              </hardware>
-              <joint name="rear_left_wheel_joint">
-                <command_interface name="velocity" />
-                <state_interface name="velocity" />
-                <state_interface name="position" />
-              </joint>
-              <joint name="rear_right_wheel_joint">
-                <command_interface name="velocity" />
-                <state_interface name="velocity" />
-                <state_interface name="position" />
-              </joint>
-              <joint name="front_left_steering_joint">
-                <command_interface name="position" />
-                <state_interface name="position" />
-              </joint>
-              <joint name="front_right_steering_joint">
-                <command_interface name="position" />
-                <state_interface name="position" />
-              </joint>
-        </xacro:if>
-        <!-- ros2_control Real Robot -->
-        <xacro:unless value="$(arg is_sim)">
-            <hardware>
-                <plugin>tamiyabot_firmware/TamiyabotInterface</plugin>
-                <param name="port">/dev/ttyACM0</param>
-            </hardware>
-        </xacro:unless>
-    </ros2_control>
+    <!-- ros2_control Gazebo -->
+    <xacro:if value="$(arg is_sim)">
+      <hardware>
+        <plugin>car_gazebo/CarlikeBotSystemHardware</plugin>
+        <param name="example_param_hw_start_duration_sec">0</param>
+        <param name="example_param_hw_stop_duration_sec">3.0</param>
+      </hardware>
+      <joint name="virtual_front_wheel_joint">
+        <command_interface name="position" />
+        <state_interface name="position" />
+      </joint>
+      <joint name="virtual_rear_wheel_joint">
+        <command_interface name="velocity" />
+        <state_interface name="velocity" />
+        <state_interface name="position" />
+      </joint>
+    </xacro:if>
+    <!-- ros2_control Real Robot -->
+    <xacro:unless value="$(arg is_sim)">
+      <hardware>
+        <plugin>tamiyabot_firmware/TamiyabotInterface</plugin>
+        <param name="port">/dev/ttyACM0</param>
+      </hardware>
+    </xacro:unless>
+  </ros2_control>
 </robot>

File: tamiyabot_description/urdf/tamiyabot_model.urdf.xacro (robot description, xacro)
@@ -6,4 +6,13 @@
   <!-- <xacro:include filename="$(find tamiyabot_description)/urdf/camera.xacro"/> -->
   <!-- <xacro:include filename="$(find tamiyabot_description)/urdf/lidar.xacro"/> -->
+  <xacro:property name="PI" value="3.1415926535897931" />
+  <xacro:property name="base_mass" value="8.0" /> <!-- arbitrary value for base mass -->
+  <xacro:property name="base_length" value="1.0" />
+  <xacro:property name="base_width" value="0.53" />
+  <xacro:property name="base_height" value="0.32" />
+  <xacro:property name="wheel_mass" value="0.1" /> <!-- arbitrary value for wheel mass -->
+  <xacro:property name="wheelbase" value="0.46" />
+  <xacro:property name="wheel_len" value="0.08" />
+  <xacro:property name="wheel_radius" value="0.047" />
   <material name="yellow">
     <color rgba="0.700 0.700 0.0 1.000"/>
@@ -181,4 +190,56 @@
   </collision>
 </link>
+<!-- rear wheels -->
+<!-- virtual rear wheel -->
+<link name="virtual_rear_wheel">
+    <visual>
+        <origin xyz="0.0 0.0 0.0" rpy="${PI/2} 0 0" />
+        <geometry>
+            <cylinder length="0.01" radius="${wheel_radius}" />
+        </geometry>
+        <material name="blue" />
+    </visual>
+    <inertial>
+    <mass value="0.1"/>  <!-- Adjust mass as needed -->
+    <inertia
+      ixx="0.001" ixy="0.0" ixz="0.0"
+      iyy="0.001" iyz="0.0"
+      izz="0.001"/>
+  </inertial>
+</link>
+<joint name="virtual_rear_wheel_joint" type="continuous">
+    <parent link="base_link" />
+    <child link="virtual_rear_wheel" />
+    <origin xyz="-0.234009 -0.032 -0.013" rpy="0 0 0" />
+    <axis xyz="0 1.0 0" />
+    <limit effort="100.0" velocity="100.0" />
+    <!-- <dynamics damping="0.2" /> -->
+</joint>
+<!-- front wheels -->
+<!-- virtual front wheel -->
+<link name="virtual_front_wheel">
+    <visual>
+        <origin xyz="0 0 0" rpy="${PI/2} 0 0.0" />
+        <geometry>
+            <cylinder length="0.01" radius="${wheel_radius}" />
+        </geometry>
+        <material name="blue" />
+    </visual>
+    <inertial>
+    <mass value="0.1"/>  <!-- Adjust mass as needed -->
+    <inertia
+      ixx="0.001" ixy="0.0" ixz="0.0"
+      iyy="0.001" iyz="0.0"
+      izz="0.001"/>
+  </inertial>
+</link>
+<joint name="virtual_front_wheel_joint" type="revolute">
+    <parent link="base_link" />
+    <child link="virtual_front_wheel" />
+    <origin xyz="0.029991 -0.032 -0.017" rpy="0 0 0.0" />
+    <axis xyz="0 0 -1" />
+    <limit lower="-0.3488" upper="0.3488" effort="100.0" velocity="0.0" />
+    <!-- <dynamics damping="0.2" /> -->
+</joint>
 <!-- Define the joints -->
 <joint name="base_joint" type="fixed">
@@ -192,4 +253,5 @@
   <child link="rear_left_wheel1"/>
   <axis xyz="0.0 1.0 0.0"/>
+  <mimic joint="virtual_rear_wheel_joint" multiplier="1.0" offset="0.0" />
 </joint>
 <joint name="rear_right_wheel_joint" type="continuous">
@@ -198,4 +260,5 @@
   <child link="rear_right_wheel1"/>
   <axis xyz="0.0 1.0 0.0"/>
+  <mimic joint="virtual_rear_wheel_joint" multiplier="1.0" offset="0.0" />
 </joint>
 <joint name="front_right_steering_joint" type="revolute">
@@ -205,4 +268,5 @@
   <axis xyz="0.0 0.0 -1.0"/>
   <limit upper="0.785398" lower="-0.785398" effort="100000" velocity="30"/>
+  <mimic joint="virtual_front_wheel_joint" multiplier="1.0" offset="0.0" />
 </joint>
 <joint name="front_left_steering_joint" type="revolute">
@@ -212,4 +276,5 @@
   <axis xyz="0.0 0.0 -1.0"/>
   <limit upper="0.785398" lower="-0.785398" effort="100000" velocity="30"/>
+  <mimic joint="virtual_front_wheel_joint" multiplier="1.0" offset="0.0" />
 </joint>
 <joint name="front_right_wheel_joint" type="continuous">

Commit message: working with odometry publish

File: tamiyabot_description/urdf/ros2_controller.xacro (robot description, xacro)
@@ -1,37 +1,37 @@
 <?xml version="1.0"?>
 <robot xmlns:xacro="http://www.ros.org/wiki/xacro" name="tamiyabot">
-     <!-- Ackermann driver -->
+  <!-- Ackermann driver -->
   <ros2_control name="RobotSystem" type="system">
-        <!-- ros2_control Gazebo -->
-        <xacro:if value="$(arg is_sim)">
-              <hardware>
-                <plugin>gz_ros2_control/GazeboSimSystem</plugin>
-              </hardware>
-              <joint name="rear_left_wheel_joint">
-                <command_interface name="velocity" />
-                <state_interface name="velocity" />
-                <state_interface name="position" />
-              </joint>
-              <joint name="rear_right_wheel_joint">
-                <command_interface name="velocity" />
-                <state_interface name="velocity" />
-                <state_interface name="position" />
-              </joint>
-              <joint name="front_left_steering_joint">
-                <command_interface name="position" />
-                <state_interface name="position" />
-              </joint>
-              <joint name="front_right_steering_joint">
-                <command_interface name="position" />
-                <state_interface name="position" />
-              </joint>
-        </xacro:if>
-        <!-- ros2_control Real Robot -->
-        <xacro:unless value="$(arg is_sim)">
-            <hardware>
-                <plugin>tamiyabot_firmware/TamiyabotInterface</plugin>
-                <param name="port">/dev/ttyACM0</param>
-            </hardware>
-        </xacro:unless>
-    </ros2_control>
+    <!-- ros2_control Gazebo -->
+    <xacro:if value="$(arg is_sim)">
+      <hardware>
+        <plugin>gz_ros2_control/GazeboSimSystem</plugin>
+      </hardware>
+      <joint name="rear_left_wheel_joint">
+        <command_interface name="velocity" />
+        <state_interface name="velocity" />
+        <state_interface name="position" />
+      </joint>
+      <joint name="rear_right_wheel_joint">
+        <command_interface name="velocity" />
+        <state_interface name="velocity" />
+        <state_interface name="position" />
+      </joint>
+      <joint name="left_wheel_steering_joint">
+        <command_interface name="position" />
+        <state_interface name="position" />
+      </joint>
+      <joint name="right_wheel_steering_joint">
+        <command_interface name="position" />
+        <state_interface name="position" />
+      </joint>
+    </xacro:if>
+    <!-- ros2_control Real Robot -->
+    <xacro:unless value="$(arg is_sim)">
+      <hardware>
+        <plugin>tamiyabot_firmware/TamiyabotInterface</plugin>
+        <param name="port">/dev/ttyACM0</param>
+      </hardware>
+    </xacro:unless>
+  </ros2_control>
 </robot>

File: tamiyabot_description/urdf/tamiyabot_gazebo.xacro (robot description, xacro)
@@ -3,29 +3,6 @@
     <gazebo>
         <plugin filename="gz_ros2_control-system" name="gz_ros2_control::GazeboSimROS2ControlPlugin">
-            <ros>
-                <remapping>tamiyabot_controller/odometry:=odom</remapping>
-                <remapping>tamiyabot_controller/tf_odometry:=tf</remapping>
-            </ros>
             <parameters>$(find tamiyabot_controller)/config/tamiyabot_controllers.yaml</parameters>
         </plugin>
-        <plugin filename="gz-sim-sensors-system" name="gz::sim::systems::Sensors">
-            <render_engine>ogre2</render_engine>
-        </plugin>
-    </gazebo>
-    <gazebo reference="front_right_wheel">
-        <mu1>1.0</mu1>
-        <mu2>1.0</mu2>
-    </gazebo>
-    <gazebo reference="front_left_wheel">
-        <mu1>1.0</mu1>
-        <mu2>1.0</mu2>
-    </gazebo>
-    <gazebo reference="rear_right_wheel">
-        <mu1>1.0</mu1>
-        <mu2>1.0</mu2>
-    </gazebo>
-    <gazebo reference="rear_left_wheel">
-        <mu1>1.0</mu1>
-        <mu2>1.0</mu2>
     </gazebo>
     <gazebo reference="laser_link">

File: tamiyabot_description/urdf/tamiyabot_model.urdf.xacro (robot description, xacro)
@@ -200,16 +200,16 @@
   <axis xyz="0.0 1.0 0.0"/>
 </joint>
-<joint name="front_right_steering_joint" type="revolute">
+<joint name="right_wheel_steering_joint" type="revolute">
   <origin xyz="0.029991 -0.1005 -0.017" rpy="0 0 0"/>
   <parent link="base_link"/>
   <child link="steering_right_link1"/>
-  <axis xyz="0.0 0.0 -1.0"/>
+  <axis xyz="0.0 0.0 1.0"/>
   <limit upper="0.785398" lower="-0.785398" effort="100" velocity="30"/>
 </joint>
-<joint name="front_left_steering_joint" type="revolute">
+<joint name="left_wheel_steering_joint" type="revolute">
   <origin xyz="0.029991 0.0365 -0.017" rpy="0 0 0"/>
   <parent link="base_link"/>
   <child link="steering_left_link1"/>
-  <axis xyz="0.0 0.0 -1.0"/>
+  <axis xyz="0.0 0.0 1.0"/>
   <limit upper="0.785398" lower="-0.785398" effort="100" velocity="30"/>
 </joint>
