Commit message: Fixed urdf, controller and remapping

File: tamiyabot_description/urdf/tamiyabot_model.urdf (Copy).xacro (robot description, xacro)
@@ -16,10 +16,10 @@
 <link name="base_link">
   <inertial>
-    <origin xyz="-0.010832508707129422 0.0 0.07339904454848215" rpy="0 0 0"/>
+    <origin xyz="-0.010832508707129422 -0.0319999966499438 0.07339904454848215" rpy="0 0 0"/>
     <mass value="37.13312619630159"/>
     <inertia ixx="0.16987923440449046" iyy="0.3219956854189482" izz="0.3110549539990225" ixy="-5.542446526035638e-09" iyz="8.55484284800756e-09" ixz="-0.054011183378953734"/>
   </inertial>
   <visual>
-    <origin xyz="0 0.03 0" rpy="0 0 0"/>
+    <origin xyz="0 0 0" rpy="0 0 0"/>
     <geometry>
       <mesh filename="package://tamiyabot_description/meshes/base_link.stl" scale="0.001 0.001 0.001"/>
@@ -29,5 +29,5 @@
   </visual>
   <collision>
-    <origin xyz="0 0.03 0" rpy="0 0 0"/>
+    <origin xyz="0 0 0" rpy="0 0 0"/>
     <geometry>
       <mesh filename="package://tamiyabot_description/meshes/base_link.stl" scale="0.001 0.001 0.001"/>
@@ -42,5 +42,5 @@
   </inertial>
   <visual>
-    <origin xyz="0.234009 -0.03 0.013" rpy="0 0 0"/>
+    <origin xyz="0.234009 -0.0155 0.013" rpy="0 0 0"/>
     <geometry>
       <mesh filename="package://tamiyabot_description/meshes/rear_left_wheel1.stl" scale="0.001 0.001 0.001"/>
@@ -50,5 +50,5 @@
   </visual>
   <collision>
-    <origin xyz="0.234009 -0.03 0.013" rpy="0 0 0"/>
+    <origin xyz="0.234009 -0.0155 0.013" rpy="0 0 0"/>
     <geometry>
       <mesh filename="package://tamiyabot_description/meshes/rear_left_wheel1.stl" scale="0.001 0.001 0.001"/>
@@ -63,5 +63,5 @@
   </inertial>
   <visual>
-    <origin xyz="0.234009 0.09 0.013" rpy="0 0 0"/>
+    <origin xyz="0.234009 0.0795 0.013" rpy="0 0 0"/>
     <geometry>
       <mesh filename="package://tamiyabot_description/meshes/rear_right_wheel1.stl" scale="0.001 0.001 0.001"/>
@@ -71,5 +71,5 @@
   </visual>
   <collision>
-    <origin xyz="0.234009 0.09 0.013" rpy="0 0 0"/>
+    <origin xyz="0.234009 0.0795 0.013" rpy="0 0 0"/>
     <geometry>
       <mesh filename="package://tamiyabot_description/meshes/rear_right_wheel1.stl" scale="0.001 0.001 0.001"/>
@@ -84,5 +84,5 @@
   </inertial>
   <visual>
-    <origin xyz="-0.026 0.1 0.017" rpy="0 0 0"/>
+    <origin xyz="-0.029991 0.1005 0.017" rpy="0 0 0"/>
     <geometry>
       <mesh filename="package://tamiyabot_description/meshes/steering_right_link1.stl" scale="0.001 0.001 0.001"/>
@@ -92,5 +92,5 @@
   </visual>
   <collision>
-    <origin xyz="-0.026 0.1 0.017" rpy="0 0 0"/>
+    <origin xyz="-0.029991 0.1005 0.017" rpy="0 0 0"/>
     <geometry>
       <mesh filename="package://tamiyabot_description/meshes/steering_right_link1.stl" scale="0.001 0.001 0.001"/>
@@ -105,5 +105,5 @@
   </inertial>
   <visual>
-    <origin xyz="-0.029991 0.095 0.013" rpy="0 0 0"/>
+    <origin xyz="-0.029991 0.1005 0.013" rpy="0 0 0"/>
     <geometry>
       <mesh filename="package://tamiyabot_description/meshes/front_right_wheel1.stl" scale="0.001 0.001 0.001"/>
@@ -113,5 +113,5 @@
   </visual>
   <collision>
-    <origin xyz="-0.029991 0.095 0.013" rpy="0 0 0"/>
+    <origin xyz="-0.029991 0.1005 0.013" rpy="0 0 0"/>
     <geometry>
       <mesh filename="package://tamiyabot_description/meshes/front_right_wheel1.stl" scale="0.001 0.001 0.001"/>
@@ -126,5 +126,5 @@
   </inertial>
   <visual>
-    <origin xyz="-0.03 -0.02 0.017" rpy="0 0 0"/>
+    <origin xyz="-0.029991 -0.0365 0.017" rpy="0 0 0"/>
     <geometry>
       <mesh filename="package://tamiyabot_description/meshes/steering_left_link1.stl" scale="0.001 0.001 0.001"/>
@@ -134,5 +134,5 @@
   </visual>
   <collision>
-    <origin xyz="-0.03 -0.02 0.017" rpy="0 0 0"/>
+    <origin xyz="-0.029991 -0.0365 0.017" rpy="0 0 0"/>
     <geometry>
       <mesh filename="package://tamiyabot_description/meshes/steering_left_link1.stl" scale="0.001 0.001 0.001"/>
@@ -147,5 +147,5 @@
   </inertial>
   <visual>
-    <origin xyz="-0.029991 -0.035 0.013" rpy="0 0 0"/>
+    <origin xyz="-0.029991 -0.0365 0.013" rpy="0 0 0"/>
     <geometry>
       <mesh filename="package://tamiyabot_description/meshes/front_left_wheel1.stl" scale="0.001 0.001 0.001"/>
@@ -155,5 +155,5 @@
   </visual>
   <collision>
-    <origin xyz="-0.029991 -0.035 0.013" rpy="0 0 0"/>
+    <origin xyz="-0.029991 -0.0365 0.013" rpy="0 0 0"/>
     <geometry>
       <mesh filename="package://tamiyabot_description/meshes/front_left_wheel1.stl" scale="0.001 0.001 0.001"/>
@@ -168,5 +168,5 @@
   </inertial>
   <visual>
-    <origin xyz="-0.059991 0.032 -0.182" rpy="0 0 0"/>
+    <origin xyz="-0.079991 0.032 -0.162" rpy="0 0 0"/>
     <geometry>
       <mesh filename="package://tamiyabot_description/meshes/Camera11.stl" scale="0.001 0.001 0.001"/>
@@ -176,5 +176,5 @@
   </visual>
   <collision>
-    <origin xyz="-0.059991 0.032 -0.182" rpy="0 0 0"/>
+    <origin xyz="-0.079991 0.032 -0.162" rpy="0 0 0"/>
     <geometry>
       <mesh filename="package://tamiyabot_description/meshes/Camera11.stl" scale="0.001 0.001 0.001"/>
@@ -186,8 +186,8 @@
     <parent link="base_footprint"/>
     <child link="base_link"/>
-    <origin xyz="0.0 0.0 0.01" rpy="0.0 0.0 0.0"/>
+    <origin xyz="0.0 0.0 0.1" rpy="0.0 0.0 0.0"/>
 </joint>
 <joint name="rear_left_wheel_joint" type="continuous">
-  <origin xyz="-0.234009 0.06 -0.013" rpy="0 0 0"/>
+  <origin xyz="-0.234009 0.0155 -0.013" rpy="0 0 0"/>
   <parent link="base_link"/>
   <child link="rear_left_wheel1"/>
@@ -195,5 +195,5 @@
 </joint>
 <joint name="rear_right_wheel_joint" type="continuous">
-  <origin xyz="-0.234009 -0.06 -0.013" rpy="0 0 0"/>
+  <origin xyz="-0.234009 -0.0795 -0.013" rpy="0 0 0"/>
   <parent link="base_link"/>
   <child link="rear_right_wheel1"/>
@@ -201,5 +201,5 @@
 </joint>
 <joint name="right_wheel_steering_joint" type="revolute">
-  <origin xyz="0.028 -0.06 -0.017" rpy="0 0 0"/>
+  <origin xyz="0.029991 -0.1005 -0.017" rpy="0 0 0"/>
   <parent link="base_link"/>
   <child link="steering_right_link1"/>
@@ -208,5 +208,5 @@
 </joint>
 <joint name="left_wheel_steering_joint" type="revolute">
-  <origin xyz="0.028 0.06 -0.017" rpy="0 0 0"/>
+  <origin xyz="0.029991 0.0365 -0.017" rpy="0 0 0"/>
   <parent link="base_link"/>
   <child link="steering_left_link1"/>
@@ -215,5 +215,5 @@
 </joint>
 <joint name="front_right_wheel_joint" type="continuous">
-  <origin xyz="0.0 0.0 0.004" rpy="0 0 0"/>
+  <origin xyz="0.0 0.01 0.004" rpy="0 0 0"/>
   <parent link="steering_right_link1"/>
   <child link="front_right_wheel1"/>
@@ -221,5 +221,5 @@
 </joint>
 <joint name="front_left_wheel_joint" type="continuous">
-  <origin xyz="0.0 0.0 0.004" rpy="0 0 0"/>
+  <origin xyz="0.0 -0.01 0.004" rpy="0 0 0"/>
   <parent link="steering_left_link1"/>
   <child link="front_left_wheel1"/>
@@ -227,5 +227,5 @@
 </joint>
 <joint name="camera_joint" type="fixed">
-  <origin xyz="0.079991 0.0 0.162" rpy="0 0.785398 0"/>
+  <origin xyz="0.079991 -0.032 0.162" rpy="0 0 0"/>
   <parent link="base_link"/>
   <child link="Camera11"/>

File: tamiyabot_description/urdf/tamiyabot_model.urdf_edited.xacro (robot description, xacro)
@@ -16,5 +16,5 @@
 <link name="base_link">
   <inertial>
-    <origin xyz="-0.010832508707129422 0.0 0.07339904454848215" rpy="0 0 0"/>
+    <origin xyz="-0.010832508707129422 -0.0319999966499438 0.07339904454848215" rpy="0 0 0"/>
     <mass value="37.13312619630159"/>
     <inertia ixx="0.16987923440449046" iyy="0.3219956854189482" izz="0.3110549539990225" ixy="-5.542446526035638e-09" iyz="8.55484284800756e-09" ixz="-0.054011183378953734"/>
@@ -84,5 +84,5 @@
   </inertial>
   <visual>
-    <origin xyz="-0.026 0.1 0.017" rpy="0 0 0"/>
+    <origin xyz="0.0 0.06 0.017" rpy="0 0 0"/>
     <geometry>
       <mesh filename="package://tamiyabot_description/meshes/steering_right_link1.stl" scale="0.001 0.001 0.001"/>
@@ -92,5 +92,5 @@
   </visual>
   <collision>
-    <origin xyz="-0.026 0.1 0.017" rpy="0 0 0"/>
+    <origin xyz="0.0 0.0 0.017" rpy="0 0 0"/>
     <geometry>
       <mesh filename="package://tamiyabot_description/meshes/steering_right_link1.stl" scale="0.001 0.001 0.001"/>
@@ -126,5 +126,5 @@
   </inertial>
   <visual>
-    <origin xyz="-0.03 -0.02 0.017" rpy="0 0 0"/>
+    <origin xyz="0.0 0.0 0.017" rpy="0 0 0"/>
     <geometry>
       <mesh filename="package://tamiyabot_description/meshes/steering_left_link1.stl" scale="0.001 0.001 0.001"/>
@@ -134,5 +134,5 @@
   </visual>
   <collision>
-    <origin xyz="-0.03 -0.02 0.017" rpy="0 0 0"/>
+    <origin xyz="0.0 0.0 0.017" rpy="0 0 0"/>
     <geometry>
       <mesh filename="package://tamiyabot_description/meshes/steering_left_link1.stl" scale="0.001 0.001 0.001"/>
@@ -168,5 +168,5 @@
   </inertial>
   <visual>
-    <origin xyz="-0.059991 0.032 -0.182" rpy="0 0 0"/>
+    <origin xyz="-0.079991 0.032 -0.162" rpy="0 0 0"/>
     <geometry>
       <mesh filename="package://tamiyabot_description/meshes/Camera11.stl" scale="0.001 0.001 0.001"/>
@@ -176,5 +176,5 @@
   </visual>
   <collision>
-    <origin xyz="-0.059991 0.032 -0.182" rpy="0 0 0"/>
+    <origin xyz="-0.079991 0.032 -0.162" rpy="0 0 0"/>
     <geometry>
       <mesh filename="package://tamiyabot_description/meshes/Camera11.stl" scale="0.001 0.001 0.001"/>
@@ -227,5 +227,5 @@
 </joint>
 <joint name="camera_joint" type="fixed">
-  <origin xyz="0.079991 0.0 0.162" rpy="0 0.785398 0"/>
+  <origin xyz="0.079991 0.0 0.162" rpy="0 0 0"/>
   <parent link="base_link"/>
   <child link="Camera11"/>
