Commit message: fix the stearing directions

File: tamiyabot_description/urdf/tamiyabot_model.urdf.xacro (robot description, xacro)
@@ -183,6 +183,6 @@
       <parent link="base_link"/>
       <child link="steering_right_link1"/>
-      <axis xyz="0.0 0.0 -1.0"/>
-      <limit effort="1000.0" lower="-0.78" upper="0.78" velocity="30"/>
+      <axis xyz="0.0 0.0 1.0"/>
+      <limit effort="1000.0" lower="-0.95" upper="0.95" velocity="30"/>
     </joint>
     <joint name="front_left_steering_joint" type="revolute">
@@ -190,6 +190,6 @@
       <parent link="base_link"/>
       <child link="steering_left_link1"/>
-      <axis xyz="0.0 0.0 -1.0"/>
-      <limit effort="1000.0" lower="-0.78" upper="0.78" velocity="30"/>
+      <axis xyz="0.0 0.0 1.0"/>
+      <limit effort="1000.0" lower="-0.95" upper="0.95" velocity="30"/>
     </joint>
     <joint name="front_right_wheel_joint" type="continuous">
@@ -203,5 +203,5 @@
       <parent link="steering_left_link1"/>
       <child link="front_left_wheel1"/>
-      <axis xyz="0.0 1.0 0.0"/>
+      <axis xyz="0.0 -1.0 0.0"/>
     </joint>
 </robot>

Commit message: Create new urdf model and fixed the missing link between base_link and front wheel

File: tamiyabot_description/urdf/tamiyabot_model.urdf.xacro (robot description, xacro)
@@ -1,207 +1,232 @@
-<?xml version="1.0"?>
+<?xml version="1.0" ?>
 <robot name="tamiyabot" xmlns:xacro="http://www.ros.org/wiki/xacro">
-  <!-- Load Simulated or Real Hardware Interfaces -->
-    <xacro:arg name="is_sim" default="true"/>
-    <xacro:include filename="$(find tamiyabot_description)/urdf/tamiyabot_gazebo.xacro"/>
-    <xacro:include filename="$(find tamiyabot_description)/urdf/ros2_controller.xacro"/>
-    <xacro:include filename="$(find tamiyabot_description)/urdf/camera.xacro"/>
-    <xacro:include filename="$(find tamiyabot_description)/urdf/lidar.xacro"/>
-    <material name="yellow">
-      <color rgba="0.700 0.700 0.0 1.000"/>
-    </material>
-    <material name="black">
-      <color rgba="0.0 0.0 0.0 1.000"/>
-    </material>
-    <link name="base_footprint"/>
-    <link name="base_link">
-      <inertial>
-        <origin xyz="0.010815142511446933 -3.80863951135197e-09 0.07339903009582542" rpy="0 0 0"/>
-        <mass value="37.13313327702305"/>
-        <inertia ixx="0.16987930061269707" iyy="0.32199575199173264" izz="0.31105499455066093" ixy="-6.034001414049238e-09" iyz="-1.2195214162965724e-08" ixz="0.05401115948790655"/>
-      </inertial>
-      <visual>
-        <origin xyz="0 0 0" rpy="0 0 0"/>
-        <geometry>
-          <mesh filename="package://tamiyabot_description/meshes/base_link.stl" scale="0.001 0.001 0.001"/>
-        </geometry>
-        <material name="yellow"/>
-        <material/>
-      </visual>
-      <collision>
-        <origin xyz="0 0 0" rpy="0 0 0"/>
-        <geometry>
-          <mesh filename="package://tamiyabot_description/meshes/base_link.stl" scale="0.001 0.001 0.001"/>
-        </geometry>
-      </collision>
-    </link>
-    <link name="rear_left_wheel1">
-      <inertial>
-        <origin xyz="3.2111828857095404e-07 -0.02099999999999999 -3.469446951953614e-18" rpy="0 0 0"/>
-        <mass value="1.805484365815081"/>
-        <inertia ixx="0.0010476743842937689" iyy="0.0015752996272436204" izz="0.0010476743842938452" ixy="1.3877787807814457e-17" iyz="-2.168404344971009e-19" ixz="-1.734723475976807e-18"/>
-      </inertial>
-      <visual>
-        <origin xyz="-0.233991 0.0475 0.013" rpy="0 0 0"/>
-        <geometry>
-          <mesh filename="package://tamiyabot_description/meshes/rear_left_wheel1.stl" scale="0.001 0.001 0.001"/>
-        </geometry>
-        <material name="black"/>
-        <material/>
-      </visual>
-      <collision>
-        <origin xyz="-0.233991 0.0475 0.013" rpy="0 0 0"/>
-        <geometry>
-          <mesh filename="package://tamiyabot_description/meshes/rear_left_wheel1.stl" scale="0.001 0.001 0.001"/>
-        </geometry>
-      </collision>
-    </link>
-    <link name="rear_right_wheel1">
-      <inertial>
-        <origin xyz="3.2111828857095404e-07 0.02099999999999999 -6.938893903907228e-18" rpy="0 0 0"/>
-        <mass value="1.805484365815081"/>
-        <inertia ixx="0.0010476743842937671" iyy="0.0015752996272436204" izz="0.0010476743842938452" ixy="-6.938893903907228e-18" iyz="-2.168404344971009e-19" ixz="8.673617379884035e-19"/>
-      </inertial>
-      <visual>
-        <origin xyz="-0.233991 -0.0475 0.013" rpy="0 0 0"/>
-        <geometry>
-          <mesh filename="package://tamiyabot_description/meshes/rear_right_wheel1.stl" scale="0.001 0.001 0.001"/>
-        </geometry>
-        <material name="black"/>
-        <material/>
-      </visual>
-      <collision>
-        <origin xyz="-0.233991 -0.0475 0.013" rpy="0 0 0"/>
-        <geometry>
-          <mesh filename="package://tamiyabot_description/meshes/rear_right_wheel1.stl" scale="0.001 0.001 0.001"/>
-        </geometry>
-      </collision>
-    </link>
-    <link name="front_right_wheel1">
-      <inertial>
-        <origin xyz="3.211182886334041e-07 -0.010465813929997403 3.469446951953614e-18" rpy="0 0 0"/>
-        <mass value="0.9105437032741223"/>
-        <inertia ixx="0.00043160993546110995" iyy="0.0007963687276588254" izz="0.0004316121960988399" ixy="0.0" iyz="4.336808689942018e-19" ixz="-5.421010862427522e-20"/>
-      </inertial>
-      <visual>
-        <origin xyz="0.030009 0.0685 0.013" rpy="0 0 0"/>
-        <geometry>
-          <mesh filename="package://tamiyabot_description/meshes/front_left_wheel1.stl" scale="0.001 0.001 0.001"/>
-        </geometry>
-        <material name="black"/>
-        <material/>
-      </visual>
-      <collision>
-        <origin xyz="0.030009 0.0685 0.013" rpy="0 0 0"/>
-        <geometry>
-          <mesh filename="package://tamiyabot_description/meshes/front_left_wheel1.stl" scale="0.001 0.001 0.001"/>
-        </geometry>
-      </collision>
-    </link>
-    <link name="front_left_wheel1">
-      <inertial>
-        <origin xyz="3.2111828862993463e-07 0.010465813929997389 3.469446951953614e-18" rpy="0 0 0"/>
-        <mass value="0.9105437032741226"/>
-        <inertia ixx="0.00043160993546111255" iyy="0.0007963687276588255" izz="0.00043161219609884425" ixy="8.673617379884035e-19" iyz="3.2526065174565133e-19" ixz="8.131516293641283e-19"/>
-      </inertial>
-      <visual>
-        <origin xyz="0.030009 -0.0685 0.013" rpy="0 0 0"/>
-        <geometry>
-          <mesh filename="package://tamiyabot_description/meshes/front_right_wheel1.stl" scale="0.001 0.001 0.001"/>
-        </geometry>
-        <material name="black"/>
-        <material/>
-      </visual>
-      <collision>
-        <origin xyz="0.030009 -0.0685 0.013" rpy="0 0 0"/>
-        <geometry>
-          <mesh filename="package://tamiyabot_description/meshes/front_right_wheel1.stl" scale="0.001 0.001 0.001"/>
-        </geometry>
-      </collision>
-    </link>
-    <link name="steering_right_link1">
-      <inertial>
-        <origin xyz="3.211182176311722e-07 0.00017084402931685783 -0.004000000028663839" rpy="0 0 0"/>
-        <mass value="0.0031874991762403456"/>
-        <inertia ixx="6.951495375836158e-08" iyy="2.9377757708371303e-08" izz="7.17755913672023e-08" ixy="-1.5094127120071632e-18" iyz="-6.094893334604098e-16" ixz="-2.117582368135751e-22"/>
-      </inertial>
-      <visual>
-        <origin xyz="0.030009 0.0685 0.009" rpy="0 0 0"/>
-        <geometry>
-          <mesh filename="package://tamiyabot_description/meshes/steering_right_link1.stl" scale="0.001 0.001 0.001"/>
-        </geometry>
-        <material name="black"/>
-        <material/>
-      </visual>
-      <collision>
-        <origin xyz="0.030009 0.0685 0.009" rpy="0 0 0"/>
-        <geometry>
-          <mesh filename="package://tamiyabot_description/meshes/steering_right_link1.stl" scale="0.001 0.001 0.001"/>
-        </geometry>
-      </collision>
-    </link>
-    <link name="steering_left_link1">
-      <inertial>
-        <origin xyz="3.211182176311722e-07 -0.00017084402931685783 -0.004000000028663839" rpy="0 0 0"/>
-        <mass value="0.0031874991762403456"/>
-        <inertia ixx="6.951495375836158e-08" iyy="2.9377757708371303e-08" izz="7.17755913672023e-08" ixy="1.5094127120071632e-18" iyz="6.094889099439362e-16" ixz="-2.117582368135751e-22"/>
-      </inertial>
-      <visual>
-        <origin xyz="0.030009 -0.0685 0.009" rpy="0 0 0"/>
-        <geometry>
-          <mesh filename="package://tamiyabot_description/meshes/steering_left_link1.stl" scale="0.001 0.001 0.001"/>
-        </geometry>
-        <material name="black"/>
-        <material/>
-      </visual>
-      <collision>
-        <origin xyz="0.030009 -0.0685 0.009" rpy="0 0 0"/>
-        <geometry>
-          <mesh filename="package://tamiyabot_description/meshes/steering_left_link1.stl" scale="0.001 0.001 0.001"/>
-        </geometry>
-      </collision>
-    </link>
-      <!-- Define the joints -->
-      <joint name="base_joint" type="fixed">
-          <parent link="base_footprint"/>
-          <child link="base_link"/>
-          <origin xyz="0.0 0.0 0.1" rpy="0.0 0.0 0.0"/>
-      </joint>
-    <joint name="rear_left_wheel_joint" type="continuous">
-      <origin xyz="0.233991 -0.0475 -0.013" rpy="0 0 0"/>
-      <parent link="base_link"/>
-      <child link="rear_left_wheel1"/>
-      <axis xyz="0.0 -1.0 0.0"/>
-    </joint>
-    <joint name="rear_right_wheel_joint" type="continuous">
-      <origin xyz="0.233991 0.0475 -0.013" rpy="0 0 0"/>
-      <parent link="base_link"/>
-      <child link="rear_right_wheel1"/>
-      <axis xyz="0.0 -1.0 0.0"/>
-    </joint>
-    <joint name="front_right_steering_joint" type="revolute">
-      <origin xyz="-0.030009 -0.0685 -0.009" rpy="0 0 0"/>
-      <parent link="base_link"/>
-      <child link="steering_right_link1"/>
-      <axis xyz="0.0 0.0 1.0"/>
-      <limit effort="1000.0" lower="-0.95" upper="0.95" velocity="30"/>
-    </joint>
-    <joint name="front_left_steering_joint" type="revolute">
-      <origin xyz="-0.030009 0.0685 -0.009" rpy="0 0 0"/>
-      <parent link="base_link"/>
-      <child link="steering_left_link1"/>
-      <axis xyz="0.0 0.0 1.0"/>
-      <limit effort="1000.0" lower="-0.95" upper="0.95" velocity="30"/>
-    </joint>
-    <joint name="front_right_wheel_joint" type="continuous">
-      <origin xyz="0.0 0.0 -0.004" rpy="0 0 0"/>
-      <parent link="steering_right_link1"/>
-      <child link="front_right_wheel1"/>
-      <axis xyz="0.0 -1.0 0.0"/>
-    </joint>
-    <joint name="front_left_wheel_joint" type="continuous">
-      <origin xyz="0.0 0.0 -0.004" rpy="0 0 0"/>
-      <parent link="steering_left_link1"/>
-      <child link="front_left_wheel1"/>
-      <axis xyz="0.0 -1.0 0.0"/>
-    </joint>
+  <xacro:arg name="is_sim" default="true"/>
+  <xacro:include filename="$(find tamiyabot_description)/urdf/tamiyabot_gazebo.xacro"/>
+  <xacro:include filename="$(find tamiyabot_description)/urdf/ros2_controller.xacro"/>
+  <!-- <xacro:include filename="$(find tamiyabot_description)/urdf/camera.xacro"/> -->
+  <!-- <xacro:include filename="$(find tamiyabot_description)/urdf/lidar.xacro"/> -->
+  <material name="yellow">
+    <color rgba="0.700 0.700 0.0 1.000"/>
+  </material>
+  <material name="black">
+    <color rgba="0.0 0.0 0.0 1.000"/>
+  </material>
+<link name="base_footprint"/>
+<link name="base_link">
+  <inertial>
+    <origin xyz="-0.010832508707129422 -0.0319999966499438 0.07339904454848215" rpy="0 0 0"/>
+    <mass value="37.13312619630159"/>
+    <inertia ixx="0.16987923440449046" iyy="0.3219956854189482" izz="0.3110549539990225" ixy="-5.542446526035638e-09" iyz="8.55484284800756e-09" ixz="-0.054011183378953734"/>
+  </inertial>
+  <visual>
+    <origin xyz="0 0 0" rpy="0 0 0"/>
+    <geometry>
+      <mesh filename="package://tamiyabot_description/meshes/base_link.stl" scale="0.001 0.001 0.001"/>
+    </geometry>
+    <material name="yellow"/>
+    <material/>
+  </visual>
+  <collision>
+    <origin xyz="0 0 0" rpy="0 0 0"/>
+    <geometry>
+      <mesh filename="package://tamiyabot_description/meshes/base_link.stl" scale="0.001 0.001 0.001"/>
+    </geometry>
+  </collision>
+</link>
+<link name="rear_left_wheel1">
+  <inertial>
+    <origin xyz="3.21118288182376e-07 0.021000000000005174 9.71445146547012e-17" rpy="0 0 0"/>
+    <mass value="1.8054843658150816"/>
+    <inertia ixx="0.0010476743842937593" iyy="0.0015752996272435787" izz="0.0010476743842937758" ixy="8.673617379884035e-18" iyz="2.0599841277224584e-18" ixz="2.6020852139652106e-18"/>
+  </inertial>
+  <visual>
+    <origin xyz="0.234009 -0.0155 0.013" rpy="0 0 0"/>
+    <geometry>
+      <mesh filename="package://tamiyabot_description/meshes/rear_left_wheel1.stl" scale="0.001 0.001 0.001"/>
+    </geometry>
+    <material name="black"/>
+    <material/>
+  </visual>
+  <collision>
+    <origin xyz="0.234009 -0.0155 0.013" rpy="0 0 0"/>
+    <geometry>
+      <mesh filename="package://tamiyabot_description/meshes/rear_left_wheel1.stl" scale="0.001 0.001 0.001"/>
+    </geometry>
+  </collision>
+</link>
+<link name="rear_right_wheel1">
+  <inertial>
+    <origin xyz="3.211182857398853e-07 -0.020999999999994814 9.8879238130678e-17" rpy="0 0 0"/>
+    <mass value="1.8054843658150797"/>
+    <inertia ixx="0.001047674384293762" iyy="0.0015752996272436204" izz="0.0010476743842938174" ixy="0.0" iyz="3.0357660829594124e-18" ixz="4.336808689942018e-18"/>
+  </inertial>
+  <visual>
+    <origin xyz="0.234009 0.0795 0.013" rpy="0 0 0"/>
+    <geometry>
+      <mesh filename="package://tamiyabot_description/meshes/rear_right_wheel1.stl" scale="0.001 0.001 0.001"/>
+    </geometry>
+    <material name="black"/>
+    <material/>
+  </visual>
+  <collision>
+    <origin xyz="0.234009 0.0795 0.013" rpy="0 0 0"/>
+    <geometry>
+      <mesh filename="package://tamiyabot_description/meshes/rear_right_wheel1.stl" scale="0.001 0.001 0.001"/>
+    </geometry>
+  </collision>
+</link>
+<link name="steering_right_link1">
+  <inertial>
+    <origin xyz="3.2111835662068655e-07 0.0001708440293172464 0.003999999971336172" rpy="0 0 0"/>
+    <mass value="0.0031874991762403456"/>
+    <inertia ixx="6.951495375837513e-08" iyy="2.9377757708371727e-08" izz="7.177559136720569e-08" ixy="1.514494909690689e-18" iyz="-6.094884864274626e-16" ixz="6.352747104407253e-22"/>
+  </inertial>
+  <visual>
+    <origin xyz="-0.029991 0.1005 0.017" rpy="0 0 0"/>
+    <geometry>
+      <mesh filename="package://tamiyabot_description/meshes/steering_right_link1.stl" scale="0.001 0.001 0.001"/>
+    </geometry>
+    <material name="black"/>
+    <material/>
+  </visual>
+  <collision>
+    <origin xyz="-0.029991 0.1005 0.017" rpy="0 0 0"/>
+    <geometry>
+      <mesh filename="package://tamiyabot_description/meshes/steering_right_link1.stl" scale="0.001 0.001 0.001"/>
+    </geometry>
+  </collision>
+</link>
+<link name="front_right_wheel1">
+  <inertial>
+    <origin xyz="3.2111828563233247e-07 -0.01046581392999707 1.5959455978986625e-16" rpy="0 0 0"/>
+    <mass value="0.9105437032741225"/>
+    <inertia ixx="0.0004316099354611056" iyy="0.000796368727658819" izz="0.0004316121960988347" ixy="7.37257477290143e-18" iyz="2.168404344971009e-18" ixz="5.800481622797449e-18"/>
+  </inertial>
+  <visual>
+    <origin xyz="-0.029991 0.1005 0.013" rpy="0 0 0"/>
+    <geometry>
+      <mesh filename="package://tamiyabot_description/meshes/front_right_wheel1.stl" scale="0.001 0.001 0.001"/>
+    </geometry>
+    <material name="black"/>
+    <material/>
+  </visual>
+  <collision>
+    <origin xyz="-0.029991 0.1005 0.013" rpy="0 0 0"/>
+    <geometry>
+      <mesh filename="package://tamiyabot_description/meshes/front_right_wheel1.stl" scale="0.001 0.001 0.001"/>
+    </geometry>
+  </collision>
+</link>
+<link name="steering_left_link1">
+  <inertial>
+    <origin xyz="3.211183591360356e-07 -0.000170844029316497 0.003999999971336172" rpy="0 0 0"/>
+    <mass value="0.003187499176240344"/>
+    <inertia ixx="6.951495375835819e-08" iyy="2.937775770836961e-08" izz="7.177559136719891e-08" ixy="-1.508989195533536e-18" iyz="6.09488062910989e-16" ixz="0.0"/>
+  </inertial>
+  <visual>
+    <origin xyz="-0.029991 -0.0365 0.017" rpy="0 0 0"/>
+    <geometry>
+      <mesh filename="package://tamiyabot_description/meshes/steering_left_link1.stl" scale="0.001 0.001 0.001"/>
+    </geometry>
+    <material name="black"/>
+    <material/>
+  </visual>
+  <collision>
+    <origin xyz="-0.029991 -0.0365 0.017" rpy="0 0 0"/>
+    <geometry>
+      <mesh filename="package://tamiyabot_description/meshes/steering_left_link1.stl" scale="0.001 0.001 0.001"/>
+    </geometry>
+  </collision>
+</link>
+<link name="front_left_wheel1">
+  <inertial>
+    <origin xyz="3.2111828832809275e-07 0.010465813929997764 1.734723475976807e-18" rpy="0 0 0"/>
+    <mass value="0.9105437032741228"/>
+    <inertia ixx="0.0004316099354611104" iyy="0.0007963687276588275" izz="0.00043161219609884295" ixy="7.37257477290143e-18" iyz="-1.0842021724855044e-19" ixz="-7.589415207398531e-19"/>
+  </inertial>
+  <visual>
+    <origin xyz="-0.029991 -0.0365 0.013" rpy="0 0 0"/>
+    <geometry>
+      <mesh filename="package://tamiyabot_description/meshes/front_left_wheel1.stl" scale="0.001 0.001 0.001"/>
+    </geometry>
+    <material name="black"/>
+    <material/>
+  </visual>
+  <collision>
+    <origin xyz="-0.029991 -0.0365 0.013" rpy="0 0 0"/>
+    <geometry>
+      <mesh filename="package://tamiyabot_description/meshes/front_left_wheel1.stl" scale="0.001 0.001 0.001"/>
+    </geometry>
+  </collision>
+</link>
+<link name="Camera11">
+  <inertial>
+    <origin xyz="-0.01999967888171309 -2.220446049250313e-16 0.020000000000000018" rpy="0 0 0"/>
+    <mass value="0.2354999999999996"/>
+    <inertia ixx="0.0001182406250000035" iyy="1.5700000000003905e-05" izz="0.0001182406249999996" ixy="-1.8973538018496328e-18" iyz="4.336808689942018e-19" ixz="4.336808689942018e-19"/>
+  </inertial>
+  <visual>
+    <origin xyz="-0.079991 0.032 -0.162" rpy="0 0 0"/>
+    <geometry>
+      <mesh filename="package://tamiyabot_description/meshes/Camera11.stl" scale="0.001 0.001 0.001"/>
+    </geometry>
+    <material name="black"/>
+    <material/>
+  </visual>
+  <collision>
+    <origin xyz="-0.079991 0.032 -0.162" rpy="0 0 0"/>
+    <geometry>
+      <mesh filename="package://tamiyabot_description/meshes/Camera11.stl" scale="0.001 0.001 0.001"/>
+    </geometry>
+  </collision>
+</link>
+<!-- Define the joints -->
+<joint name="base_joint" type="fixed">
+    <parent link="base_footprint"/>
+    <child link="base_link"/>
+    <origin xyz="0.0 0.0 0.1" rpy="0.0 0.0 0.0"/>
+</joint>
+<joint name="rear_left_wheel_joint" type="continuous">
+  <origin xyz="-0.234009 0.0155 -0.013" rpy="0 0 0"/>
+  <parent link="base_link"/>
+  <child link="rear_left_wheel1"/>
+  <axis xyz="0.0 1.0 0.0"/>
+</joint>
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
Commit message: Updated inertia values, added relay for controller topics

File: tamiyabot_description/urdf/tamiyabot_model.urdf.xacro (robot description, xacro)
@@ -37,5 +37,8 @@
 <link name="rear_left_wheel1">
   <inertial>
+<!--
     <origin xyz="3.21118288182376e-07 0.021000000000005174 9.71445146547012e-17" rpy="0 0 0"/>
+-->
+    <origin xyz="3.21118288182376e-07 0.0081000000000005174 9.71445146547012e-17" rpy="0 0 0"/>
     <mass value="1.8054843658150816"/>
     <inertia ixx="0.0010476743842937593" iyy="0.0015752996272435787" izz="0.0010476743842937758" ixy="8.673617379884035e-18" iyz="2.0599841277224584e-18" ixz="2.6020852139652106e-18"/>
@@ -58,5 +61,5 @@
 <link name="rear_right_wheel1">
   <inertial>
-    <origin xyz="3.211182857398853e-07 -0.020999999999994814 9.8879238130678e-17" rpy="0 0 0"/>
+    <origin xyz="3.211182857398853e-07 -0.0085000000000005174 9.8879238130678e-17" rpy="0 0 0"/>
     <mass value="1.8054843658150797"/>
     <inertia ixx="0.001047674384293762" iyy="0.0015752996272436204" izz="0.0010476743842938174" ixy="0.0" iyz="3.0357660829594124e-18" ixz="4.336808689942018e-18"/>
@@ -100,5 +103,5 @@
 <link name="front_right_wheel1">
   <inertial>
-    <origin xyz="3.2111828563233247e-07 0.0 1.5959455978986625e-16" rpy="0 0 0"/>
+    <origin xyz="3.2111828563233247e-07 -0.016 1.5959455978986625e-16" rpy="0 0 0"/>
     <mass value="0.9105437032741225"/>
     <inertia ixx="0.0004316099354611056" iyy="0.000796368727658819" izz="0.0004316121960988347" ixy="7.37257477290143e-18" iyz="2.168404344971009e-18" ixz="5.800481622797449e-18"/>
@@ -142,5 +145,5 @@
 <link name="front_left_wheel1">
   <inertial>
-    <origin xyz="3.2111828832809275e-07 0.0 1.734723475976807e-18" rpy="0 0 0"/>
+    <origin xyz="3.2111828832809275e-07 0.012 1.734723475976807e-18" rpy="0 0 0"/>
     <mass value="0.9105437032741228"/>
     <inertia ixx="0.0004316099354611104" iyy="0.0007963687276588275" izz="0.00043161219609884295" ixy="7.37257477290143e-18" iyz="-1.0842021724855044e-19" ixz="-7.589415207398531e-19"/>

Commit message: Revert back joint rotation negation

File: tamiyabot_description/urdf/tamiyabot_model.urdf.xacro (robot description, xacro)
@@ -207,5 +207,5 @@
   <parent link="base_link"/>
   <child link="steering_right_link1"/>
-  <axis xyz="0.0 0.0 -1.0"/>
+  <axis xyz="0.0 0.0 1.0"/>
   <limit upper="0.785398" lower="-0.785398" effort="100" velocity="30"/>
 </joint>
@@ -214,5 +214,5 @@
   <parent link="base_link"/>
   <child link="steering_left_link1"/>
-  <axis xyz="0.0 0.0 -1.0"/>
+  <axis xyz="0.0 0.0 1.0"/>
   <limit upper="0.785398" lower="-0.785398" effort="100" velocity="30"/>
 </joint>
